File: Pinguino_SMD-4550.sch (KiCad schematic (older format))
At the start: 51 parts, among them P1 uUSB, P10 CONN_01X01, P11 CONN_01X01, P12 CONN_01X01, P13 CONN_01X01, P14 CONN_01X01, P15 CONN_01X01, P16 CONN_01X01, P17 CONN_01X01, P18 CONN_01X01, P19 CONN_01X01, P2 CONN_01X01, P20 CONN_01X01, P21 CONN_01X01, P22 CONN_01X01, P23 CONN_01X01, P24 CONN_01X01, P25 CONN_01X01, P26 CONN_01X01, P27 CONN_01X01, P28 CONN_01X01, P29 CONN_01X01, P3 CONN_01X01, P30 CONN_01X01, P31 CONN_01X01, P32 CONN_01X01, P33 CONN_01X01, P34 CONN_01X01, P35 CONN_01X01, P36 CONN_01X01, P37 CONN_01X01, P38 CONN_01X01, P4 CONN_01X01, P5 CONN_01X01, P6 CONN_01X01, P7 CONN_01X01, P8 CONN_01X01, P9 CONN_01X01, SW1 Reset, U1 PIC18(L)F4550-I/PT, Y1 Crystal

Commit message: Reorganized and aligned components.
Parts:
- added P39, P40, P41: CONN_01X01, Socket_Strips:Socket_Strip_Straight_1x01, symbol CONN_01X01
- C1, C2, C3, C4: footprint Capacitors_SMD:C_1206 -> Capacitors_SMD:C_0805
- C5: footprint Capacitors_SMD:c_elec_6.3x5.3 -> Capacitors_Tantalum_SMD:CP_Tantalum_Case-B_EIA-3528-21_Reflow
- D1, D2: footprint LEDs:LED_1206 -> LEDs:LED_0805
- R1, R2, R3: footprint Resistors_SMD:R_1206 -> Resistors_SMD:R_0805
Connections:
- net GND: now also P39.1 (P1), P40.1 (P1)
- net VCC: now also P41.1 (P1)
Changed lines of the file:
@@
 F 0 "R2" V 7480 3800 50  0000 C CNN
 F 1 "10k" V 7400 3800 50  0000 C CNN
-F 2 "Resistors_SMD:R_1206" V 7330 3800 50  0001 C CNN
+F 2 "Resistors_SMD:R_0805" V 7330 3800 50  0001 C CNN
 F 3 "" H 7400 3800 50  0000 C CNN
 	1    7400 3800
@@
 	7250 3800 7050 3800
 $Comp
-L VCC #PWR01
+L VCC #PWR18
 U 1 1 5846045B
 P 7700 3800
-F 0 "#PWR01" H 7700 3650 50  0001 C CNN
+F 0 "#PWR18" H 7700 3650 50  0001 C CNN
 F 1 "VCC" H 7700 3950 50  0000 C CNN
 F 2 "" H 7700 3800 50  0000 C CNN
@@
 	7550 4150 7750 4150
 $Comp
-L GND #PWR02
+L GND #PWR19
 U 1 1 584604D7
 P 7750 4150
-F 0 "#PWR02" H 7750 3900 50  0001 C CNN
+F 0 "#PWR19" H 7750 3900 50  0001 C CNN
 F 1 "GND" H 7750 4000 50  0000 C CNN
 F 2 "" H 7750 4150 50  0000 C CNN
@@
 F 0 "R1" V 1880 1300 50  0000 C CNN
 F 1 "470" V 1800 1300 50  0000 C CNN
-F 2 "Resistors_SMD:R_1206" V 1730 1300 50  0001 C CNN
+F 2 "Resistors_SMD:R_0805" V 1730 1300 50  0001 C CNN
 F 3 "" H 1800 1300 50  0000 C CNN
 	1    1800 1300
@@
 F 0 "D1" H 1350 1400 50  0000 C CNN
 F 1 "Run_LED" H 1350 1200 50  0000 C CNN
-F 2 "LEDs:LED_1206" H 1350 1300 50  0001 C CNN
+F 2 "LEDs:LED_0805" H 1350 1300 50  0001 C CNN
 F 3 "" H 1350 1300 50  0000 C CNN
 	1    1350 1300
@@
 $EndComp
 $Comp
-L VCC #PWR03
+L VCC #PWR4
 U 1 1 5846070F
 P 1050 1300
-F 0 "#PWR03" H 1050 1150 50  0001 C CNN
+F 0 "#PWR4" H 1050 1150 50  0001 C CNN
 F 1 "VCC" H 1050 1450 50  0000 C CNN
 F 2 "" H 1050 1300 50  0000 C CNN
@@
 F 0 "C1" H 1625 2150 50  0000 L CNN
 F 1 "22uF" V 1750 1900 50  0000 L CNN
-F 2 "Capacitors_SMD:C_1206" H 1638 1900 50  0001 C CNN
+F 2 "Capacitors_SMD:C_0805" H 1638 1900 50  0001 C CNN
 F 3 "" H 1600 2050 50  0000 C CNN
 	1    1600 2050
@@
 F 0 "C2" H 1625 2650 50  0000 L CNN
 F 1 "22uF" V 1450 2500 50  0000 L CNN
-F 2 "Capacitors_SMD:C_1206" H 1638 2400 50  0001 C CNN
+F 2 "Capacitors_SMD:C_0805" H 1638 2400 50  0001 C CNN
 F 3 "" H 1600 2550 50  0000 C CNN
 	1    1600 2550
@@
 	1750 2550 1750 2450
 $Comp
-L GND #PWR04
+L GND #PWR8
 U 1 1 584609F8
 P 1350 2050
-F 0 "#PWR04" H 1350 1800 50  0001 C CNN
+F 0 "#PWR8" H 1350 1800 50  0001 C CNN
 F 1 "GND" H 1350 1900 50  0000 C CNN
 F 2 "" H 1350 2050 50  0000 C CNN
@@
 $EndComp
 $Comp
-L GND #PWR05
+L GND #PWR9
 U 1 1 58460B40
 P 1350 2550
-F 0 "#PWR05" H 1350 2300 50  0001 C CNN
+F 0 "#PWR9" H 1350 2300 50  0001 C CNN
 F 1 "GND" H 1350 2400 50  0000 C CNN
 F 2 "" H 1350 2550 50  0000 C CNN
@@
 Connection ~ 1750 2100
 $Comp
-L VCC #PWR06
+L VCC #PWR12
 U 1 1 5846108D
 P 4400 900
-F 0 "#PWR06" H 4400 750 50  0001 C CNN
+F 0 "#PWR12" H 4400 750 50  0001 C CNN
 F 1 "VCC" H 4400 1050 50  0000 C CNN
 F 2 "" H 4400 900 50  0000 C CNN
@@
 $EndComp
 $Comp
-L GND #PWR07
+L GND #PWR13
 U 1 1 58461476
 P 4400 4300
-F 0 "#PWR07" H 4400 4050 50  0001 C CNN
+F 0 "#PWR13" H 4400 4050 50  0001 C CNN
 F 1 "GND" H 4400 4150 50  0000 C CNN
 F 2 "" H 4400 4300 50  0000 C CNN
@@
 F 0 "C4" H 7325 2500 50  0000 L CNN
 F 1 "220nF" H 7325 2300 50  0000 L CNN
-F 2 "Capacitors_SMD:C_1206" H 7338 2250 50  0001 C CNN
+F 2 "Capacitors_SMD:C_0805" H 7338 2250 50  0001 C CNN
 F 3 "" H 7300 2400 50  0000 C CNN
 	1    7300 2400
@@
 	7450 2400 7550 2400
 $Comp
-L GND #PWR08
+L GND #PWR17
 U 1 1 58464103
 P 7550 2400
-F 0 "#PWR08" H 7550 2150 50  0001 C CNN
+F 0 "#PWR17" H 7550 2150 50  0001 C CNN
 F 1 "GND" H 7550 2250 50  0000 C CNN
 F 2 "" H 7550 2400 50  0000 C CNN
@@
 F 0 "C3" H 4560 1320 50  0000 L CNN
 F 1 "100nF" V 4450 1150 50  0000 L CNN
-F 2 "Capacitors_SMD:C_1206" H 4550 1250 50  0001 C CNN
+F 2 "Capacitors_SMD:C_0805" H 4550 1250 50  0001 C CNN
 F 3 "" H 4550 1250 50  0000 C CNN
 	1    4550 1250
@@
 	7100 1900 7050 1900
 $Comp
-L VCC #PWR09
+L VCC #PWR16
 U 1 1 584662AB
 P 7050 2100
-F 0 "#PWR09" H 7050 1950 50  0001 C CNN
+F 0 "#PWR16" H 7050 1950 50  0001 C CNN
 F 1 "VCC" H 7050 2250 50  0000 C CNN
 F 2 "" H 7050 2100 50  0000 C CNN
@@
 F 0 "D2" H 8750 1850 50  0000 C CNN
 F 1 "Power_LED" H 8750 1650 50  0000 C CNN
-F 2 "LEDs:LED_1206" H 8750 1750 50  0001 C CNN
+F 2 "LEDs:LED_0805" H 8750 1750 50  0001 C CNN
 F 3 "" H 8750 1750 50  0000 C CNN
 	1    8750 1750
@@
 F 0 "R3" V 8830 2150 50  0000 C CNN
 F 1 "470" V 8750 2150 50  0000 C CNN
-F 2 "Resistors_SMD:R_1206" V 8680 2150 50  0001 C CNN
+F 2 "Resistors_SMD:R_0805" V 8680 2150 50  0001 C CNN
 F 3 "" H 8750 2150 50  0000 C CNN
 	1    8750 2150
@@
 F 0 "C5" H 9175 2000 50  0000 L CNN
 F 1 "10-100uF" V 9050 1750 50  0000 L CNN
-F 2 "Capacitors_SMD:c_elec_6.3x5.3" H 9188 1750 50  0001 C CNN
+F 2 "Capacitors_Tantalum_SMD:CP_Tantalum_Case-B_EIA-3528-21_Reflow" H 9188 1750 50  0001 C CNN
 F 3 "" H 9150 1900 50  0000 C CNN
 	1    9150 1900
@@
 $EndComp
 $Comp
-L GND #PWR010
+L GND #PWR21
 U 1 1 58466D61
 P 8750 2350
-F 0 "#PWR010" H 8750 2100 50  0001 C CNN
+F 0 "#PWR21" H 8750 2100 50  0001 C CNN
 F 1 "GND" H 8750 2200 50  0000 C CNN
 F 2 "" H 8750 2350 50  0000 C CNN
@@
 $EndComp
 $Comp
-L GND #PWR011
+L GND #PWR23
 U 1 1 58466DE1
 P 9150 2350
-F 0 "#PWR011" H 9150 2100 50  0001 C CNN
+F 0 "#PWR23" H 9150 2100 50  0001 C CNN
 F 1 "GND" H 9150 2200 50  0000 C CNN
 F 2 "" H 9150 2350 50  0000 C CNN
@@
 $EndComp
 $Comp
-L VCC #PWR012
+L VCC #PWR20
 U 1 1 58466E81
 P 8750 1500
-F 0 "#PWR012" H 8750 1350 50  0001 C CNN
+F 0 "#PWR20" H 8750 1350 50  0001 C CNN
 F 1 "VCC" H 8750 1650 50  0000 C CNN
 F 2 "" H 8750 1500 50  0000 C CNN
@@
 $EndComp
 $Comp
-L VCC #PWR013
+L VCC #PWR22
 U 1 1 58466EB1
 P 9150 1500
-F 0 "#PWR013" H 9150 1350 50  0001 C CNN
+F 0 "#PWR22" H 9150 1350 50  0001 C CNN
 F 1 "VCC" H 9150 1650 50  0000 C CNN
 F 2 "" H 9150 1500 50  0000 C CNN
@@
 	9150 2350 9150 2050
 $Comp
-L GND #PWR014
+L GND #PWR24
 U 1 1 58467238
 P 9900 1600
-F 0 "#PWR014" H 9900 1350 50  0001 C CNN
+F 0 "#PWR24" H 9900 1350 50  0001 C CNN
 F 1 "GND" H 9900 1450 50  0000 C CNN
 F 2 "" H 9900 1600 50  0000 C CNN
@@
 $EndComp
 $Comp
-L PWR_FLAG #FLG015
+L PWR_FLAG #FLG1
 U 1 1 58467268
 P 9900 1400
-F 0 "#FLG015" H 9900 1495 50  0001 C CNN
+F 0 "#FLG1" H 9900 1495 50  0001 C CNN
 F 1 "PWR_FLAG" H 9900 1580 50  0000 C CNN
 F 2 "" H 9900 1400 50  0000 C CNN
@@
 PIN28
 $Comp
-L VCC #PWR016
+L VCC #PWR10
 U 1 1 5849F271
 P 1350 5300
-F 0 "#PWR016" H 1350 5150 50  0001 C CNN
+F 0 "#PWR10" H 1350 5150 50  0001 C CNN
 F 1 "VCC" H 1350 5450 50  0000 C CNN
 F 2 "" H 1350 5300 50  0000 C CNN
@@
 $EndComp
 $Comp
-L VCC #PWR017
+L VCC #PWR6
 U 1 1 5849F2E1
 P 1150 5300
-F 0 "#PWR017" H 1150 5150 50  0001 C CNN
+F 0 "#PWR6" H 1150 5150 50  0001 C CNN
 F 1 "VCC" H 1150 5450 50  0000 C CNN
 F 2 "" H 1150 5300 50  0000 C CNN
@@
 $EndComp
 $Comp
-L GND #PWR018
+L GND #PWR11
 U 1 1 5849F351
 P 1500 6250
-F 0 "#PWR018" H 1500 6000 50  0001 C CNN
+F 0 "#PWR11" H 1500 6000 50  0001 C CNN
 F 1 "GND" H 1500 6100 50  0000 C CNN
 F 2 "" H 1500 6250 50  0000 C CNN
@@
 $EndComp
 $Comp
-L GND #PWR019
+L GND #PWR7
 U 1 1 5849F3C1
 P 1300 6250
-F 0 "#PWR019" H 1300 6000 50  0001 C CNN
+F 0 "#PWR7" H 1300 6000 50  0001 C CNN
 F 1 "GND" H 1300 6100 50  0000 C CNN
 F 2 "" H 1300 6250 50  0000 C CNN
@@
 $EndComp
 $Comp
-L GND #PWR020
+L GND #PWR5
 U 1 1 58630752
 P 1100 6250
-F 0 "#PWR020" H 1100 6000 50  0001 C CNN
+F 0 "#PWR5" H 1100 6000 50  0001 C CNN
 F 1 "GND" H 1100 6100 50  0000 C CNN
 F 2 "" H 1100 6250 50  0000 C CNN
@@
 	1100 6150 1100 6250
 $Comp
-L GND #PWR021
+L GND #PWR15
 U 1 1 58652F75
 P 7000 1700
-F 0 "#PWR021" H 7000 1450 50  0001 C CNN
+F 0 "#PWR15" H 7000 1450 50  0001 C CNN
 F 1 "GND" H 7000 1550 50  0000 C CNN
 F 2 "" H 7000 1700 50  0000 C CNN
@@
 Connection ~ 7050 1700
 $Comp
-L GND #PWR022
+L GND #PWR14
 U 1 1 586567B0
 P 4700 1250
-F 0 "#PWR022" H 4700 1000 50  0001 C CNN
+F 0 "#PWR14" H 4700 1000 50  0001 C CNN
 F 1 "GND" H 4700 1100 50  0000 C CNN
 F 2 "" H 4700 1250 50  0000 C CNN
@@
 Wire Wire Line
 	4650 1250 4700 1250
+$Comp
+L CONN_01X01 P40
+U 1 1 58ACED38
+P 900 5950
+F 0 "P40" H 900 6050 50  0000 C CNN
+F 1 "CONN_01X01" V 1000 5950 50  0001 C CNN
+F 2 "Socket_Strips:Socket_Strip_Straight_1x01" H 900 5950 50  0001 C CNN
+F 3 "" H 900 5950 50  0000 C CNN
+	1    900  5950
+	0    -1   -1   0
+$EndComp
+$Comp
+L CONN_01X01 P39
+U 1 1 58ACEDE8
+P 700 5950
+F 0 "P39" H 700 6050 50  0000 C CNN
+F 1 "CONN_01X01" V 800 5950 50  0001 C CNN
+F 2 "Socket_Strips:Socket_Strip_Straight_1x01" H 700 5950 50  0001 C CNN
+F 3 "" H 700 5950 50  0000 C CNN
+	1    700  5950
+	0    -1   -1   0
+$EndComp
+$Comp
+L GND #PWR1
+U 1 1 58ACEE68
+P 700 6250
+F 0 "#PWR1" H 700 6000 50  0001 C CNN
+F 1 "GND" H 700 6100 50  0000 C CNN
+F 2 "" H 700 6250 50  0000 C CNN
+F 3 "" H 700 6250 50  0000 C CNN
+	1    700  6250
+	1    0    0    -1
+$EndComp
+$Comp
+L GND #PWR2
+U 1 1 58ACEEE6
+P 900 6250
+F 0 "#PWR2" H 900 6000 50  0001 C CNN
+F 1 "GND" H 900 6100 50  0000 C CNN
+F 2 "" H 900 6250 50  0000 C CNN
+F 3 "" H 900 6250 50  0000 C CNN
+	1    900  6250
+	1    0    0    -1
+$EndComp
+Wire Wire Line
+	700  6150 700  6250
+Wire Wire Line
+	900  6150 900  6250
+$Comp
+L CONN_01X01 P41
+U 1 1 58ACF1C6
+P 950 5600
+F 0 "P41" H 950 5700 50  0000 C CNN
+F 1 "CONN_01X01" V 1050 5600 50  0001 C CNN
+F 2 "Socket_Strips:Socket_Strip_Straight_1x01" H 950 5600 50  0001 C CNN
+F 3 "" H 950 5600 50  0000 C CNN
+	1    950  5600
+	0    1    1    0
+$EndComp
+$Comp
+L VCC #PWR3
+U 1 1 58ACF24C
+P 950 5300
+F 0 "#PWR3" H 950 5150 50  0001 C CNN
+F 1 "VCC" H 950 5450 50  0000 C CNN
+F 2 "" H 950 5300 50  0000 C CNN
+F 3 "" H 950 5300 50  0000 C CNN
+	1    950  5300
+	1    0    0    -1
+$EndComp
+Wire Wire Line
+	950  5300 950  5400
 $EndSCHEMATC

Commit message: Reorganized and aligned components.
Connections:
- net GND: no longer P39.1 (P1)
- net ICPORTS: now reaches U1.34 ((ICPORTS))
- net ICPORTS: now also P39.1 (P1)
- no-connect marks 2 -> 1
Other:
- moved on the sheet: P39
Changed lines of the file:
@@
 Text Label 2900 3600 2    60   ~ 0
 ICSP_PGD
-NoConn ~ 3150 3700
-Wire Wire Line
-	3250 3700 3150 3700
+Wire Wire Line
+	2900 3700 3250 3700
 $Comp
 L CONN_01X01 P6
@@
 L CONN_01X01 P39
 U 1 1 58ACEDE8
-P 700 5950
-F 0 "P39" H 700 6050 50  0000 C CNN
-F 1 "CONN_01X01" V 800 5950 50  0001 C CNN
-F 2 "Socket_Strips:Socket_Strip_Straight_1x01" H 700 5950 50  0001 C CNN
-F 3 "" H 700 5950 50  0000 C CNN
-	1    700  5950
-	0    -1   -1   0
-$EndComp
-$Comp
-L GND #PWR1
-U 1 1 58ACEE68
-P 700 6250
-F 0 "#PWR1" H 700 6000 50  0001 C CNN
-F 1 "GND" H 700 6100 50  0000 C CNN
-F 2 "" H 700 6250 50  0000 C CNN
-F 3 "" H 700 6250 50  0000 C CNN
-	1    700  6250
-	1    0    0    -1
+P 4900 6200
+F 0 "P39" H 4900 6300 50  0000 C CNN
+F 1 "CONN_01X01" V 5000 6200 50  0001 C CNN
+F 2 "Socket_Strips:Socket_Strip_Straight_1x01" H 4900 6200 50  0001 C CNN
+F 3 "" H 4900 6200 50  0000 C CNN
+	1    4900 6200
+	-1   0    0    1
 $EndComp
 $Comp
@@
 $EndComp
 Wire Wire Line
-	700  6150 700  6250
-Wire Wire Line
 	900  6150 900  6250
 $Comp
@@
 Wire Wire Line
 	950  5300 950  5400
+Text Label 2900 3700 2    60   ~ 0
+ICPORTS
+Text Label 5100 6200 0    60   ~ 0
+ICPORTS
 $EndSCHEMATC

Commit message: Bug Fixed: RA4
Parts:
- C1, C2: value 22uF -> 22pF
Connections:
- net PIN17/A4: now also U1.24 (RA5/AN4/~SS~/HLVDIN/C2OUT); no longer U1.23 (RA4/T0CKI/C1OUT/RCV)
- net RA4: now also U1.23 (RA4/T0CKI/C1OUT/RCV); no longer U1.24 (RA5/AN4/~SS~/HLVDIN/C2OUT)
Changed lines of the file:
@@
 Title "Pinguino_SMD-4550"
 Date ""
-Rev "2.0"
+Rev "2.1"
 Comp "Rottdevel"
 Comment1 "Hakerspace"
@@
 P 1600 2050
 F 0 "C1" H 1625 2150 50  0000 L CNN
-F 1 "22uF" V 1750 1900 50  0000 L CNN
+F 1 "22pF" V 1750 1900 50  0000 L CNN
 F 2 "Capacitors_SMD:C_0805" H 1638 1900 50  0001 C CNN
 F 3 "" H 1600 2050 50  0000 C CNN
@@
 P 1600 2550
 F 0 "C2" H 1625 2650 50  0000 L CNN
-F 1 "22uF" V 1450 2500 50  0000 L CNN
+F 1 "22pF" V 1450 2500 50  0000 L CNN
 F 2 "Capacitors_SMD:C_0805" H 1638 2400 50  0001 C CNN
 F 3 "" H 1600 2550 50  0000 C CNN
@@
 Wire Wire Line
 	7100 2100 7050 2100
-Text Label 2900 2100 2    60   ~ 0
+Text Label 2900 2000 2    60   ~ 0
 RA4
 Wire Wire Line
@@
 Text Label 2900 1900 2    60   ~ 0
 PIN16/A3
-Text Label 2900 2000 2    60   ~ 0
+Text Label 2900 2100 2    60   ~ 0
 PIN17/A4
 Wire Wire Line
